File: nfc-ble-reader_case/nfc-ble-reader/nfc-ble-reader.kicad_pcb (KiCad board)
At the start: 2 copper layers, 90 x 70 mm, 16 parts, among them M3 MountingHole, M6 MountingHole, SW2 MK-12D13G4-B, U1 DW03C, U2 PN532_NFC_Elechouse_HW147_SPI, U3 ProMicro_NRF52840

Commit message: finalized first pcb design and ordered 10 PCBs and components for 20 devices and 100 batteries
Parts:
- renumbered M3 to H1, M3 to H2, M6 to H3, M6 to H4
Routing:
- net GND: track 7.81 -> 0.41 mm
- added copper zone on F.Cu, net GND
Changed lines of the file:
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@@
 		(descr "Mounting Hole 6.4mm, M6, no annular, generated by kicad-footprint-generator mountinghole.py")
 		(tags "mountinghole M6")
-		(property "Reference" "M6"
+		(property "Reference" "H4"
 			(at 0 4.24 0)
 			(layer "F.SilkS")
@@
 		(descr "Mounting Hole 6.4mm, M6, no annular, generated by kicad-footprint-generator mountinghole.py")
 		(tags "mountinghole M6")
-		(property "Reference" "M6"
+		(property "Reference" "H3"
 			(at 0 4.22 0)
 			(layer "F.SilkS")
@@
 		(descr "Mounting Hole 3.2mm, M3, no annular, generated by kicad-footprint-generator mountinghole.py")
 		(tags "mountinghole M3")
-		(property "Reference" "M3"
+		(property "Reference" "H1"
 			(at 0.1 2.7 0)
 			(layer "F.SilkS")
@@
 			)
 		)
+		(property "LCSC Part" "C42380663"
+			(at 0 0 0)
+			(unlocked yes)
+			(layer "F.Fab")
+			(hide yes)
+			(effects
+				(font
+					(size 1 1)
+					(thickness 0.15)
+				)
+			)
+		)
 		(sheetname "/")
 		(sheetfile "nfc-ble-reader.kicad_sch")
@@
 			)
 		)
+		(property "LCSC Part" "C2907302"
+			(at 0 0 270)
+			(unlocked yes)
+			(layer "F.Fab")
+			(hide yes)
+			(effects
+				(font
+					(size 1 1)
+					(thickness 0.15)
+				)
+			)
+		)
 		(property ki_fp_filters "R_*")
 		(sheetname "/")
@@
 			)
 		)
+		(property "LCSC Part" "C2907302"
+			(at 0 0 270)
+			(unlocked yes)
+			(layer "F.Fab")
+			(hide yes)
+			(effects
+				(font
+					(size 1 1)
+					(thickness 0.15)
+				)
+			)
+		)
 		(property ki_fp_filters "R_*")
 		(sheetname "/")
@@
 			)
 		)
+		(property "LCSC Part" "C2907232"
+			(at 0 0 270)
+			(unlocked yes)
+			(layer "F.Fab")
+			(hide yes)
+			(effects
+				(font
+					(size 1 1)
+					(thickness 0.15)
+				)
+			)
+		)
 		(property ki_fp_filters "R_*")
 		(sheetname "/")
@@
 		(descr "Mounting Hole 3.2mm, M3, no annular, generated by kicad-footprint-generator mountinghole.py")
 		(tags "mountinghole M3")
-		(property "Reference" "M3"
+		(property "Reference" "H2"
 			(at 0.1 2.7 0)
 			(layer "F.SilkS")
@@
 			)
 		)
+		(property "LCSC Part" "C46653"
+			(at 0 0 270)
+			(unlocked yes)
+			(layer "F.Fab")
+			(hide yes)
+			(effects
+				(font
+					(size 1 1)
+					(thickness 0.15)
+				)
+			)
+		)
 		(property ki_fp_filters "C_*")
 		(sheetname "/")
@@
 	)
 	(segment
-		(start 170 79)
-		(end 168.7 79)
-		(width 0.2)
-		(layer "F.Cu")
-		(net "GND")
-	)
-	(segment
-		(start 182.35 82.95)
-		(end 182.35 82.05)
-		(width 0.2)
-		(layer "F.Cu")
-		(net "GND")
-	)
-	(segment
 		(start 182.35 84.15)
 		(end 182.4 84.2)
@@
 	)
 	(segment
-		(start 170 79)
-		(end 170 80.2)
-		(width 0.2)
-		(layer "F.Cu")
-		(net "GND")
-	)
-	(segment
-		(start 182.35 82.95)
-		(end 183.75 82.95)
-		(width 0.2)
-		(layer "F.Cu")
-		(net "GND")
-	)
-	(segment
-		(start 182.35 82.95)
-		(end 182.35 84.15)
-		(width 0.2)
-		(layer "F.Cu")
-		(net "GND")
-	)
-	(segment
-		(start 170 79)
-		(end 171.4 79)
-		(width 0.2)
-		(layer "F.Cu")
-		(net "GND")
-	)
-	(segment
 		(start 182.35 82.05)
 		(end 182.4 82)
@@
 	(zone
 		(net "GND")
-		(layer "B.Cu")
+		(layers "F.Cu" "B.Cu")
 		(hatch edge 0.5)
 		(connect_pads
