File: nfc-ble-reader_case/nfc-ble-reader/nfc-ble-reader.kicad_pcb (KiCad board)
At the start: 2 copper layers, 90 x 70 mm, 16 parts, among them SW2 MK-12D13G4-B, U1 DW03C, U2 PN532_NFC_Elechouse_HW147_SPI, U3 ProMicro_NRF52840

Commit message: New licenses mandanten kompatibel Artikel verwaltung immer sichtbar Code graph neuere doku Testfälle
Parts:
- removed kibuzzard-6A8E2C3E: G***, kibuzzard-6A8E2C3E
- added kibuzzard-6ACBD38F: G***, kibuzzard-6ACBD38F, F.Cu at (160.0, 111.0)
- turned BT1 to -90 degrees
